File: Backplate-PCB/_autosave-Reversal.kicad_pcb (KiCad board)
At the start: 2 copper layers, 217.2 x 127.2 mm, 5 parts

Commit message: Initial push with stuff
Parts:
- moved REF** 12.1 mm to (33.3, 27.9)
- moved REF** 12.0 mm to (33.2, 155.6)
- moved REF** 11.5 mm to (267.8, 28.1)
- moved REF** 11.4 mm to (267.9, 155.8)
- moved G*** 0.06 mm to (150.5, 88.0)
Other:
- board size 217.2 x 127.2 mm -> 240.2 x 133.2 mm
