File: PCB_Kicad/Reversal.kicad_pcb (KiCad board)
At the start: 2 copper layers, 210 x 120 mm, 59 parts, among them J1 USB_A, SW1 SW_Push, SW10 SW_Push, SW11 SW_Push, SW12 SW_Push, SW13 SW_Push, SW14 SW_Push, SW15 SW_Push, SW16 SW_Push, SW17 SW_Push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

Commit message: Initial push with stuff
Routing:
- net GND: track 76.1 -> 167.2 mm, vias 27 -> 28
